File: RTU_Agro_new/RTU_Agro_new.kicad_sch (KiCad schematic)
At the start: 113 parts, among them IC1 STM32F103R8T6, J1 520425-3, U1 XL4015, U10 DRV8251ADDAR, U11 DRV8251ADDAR, U12 DRV8251ADDAR, U13 PCF8574T, U2 MAX3485ESA+, U3 LTC2943IDD#TRPBF, U4 M24128-BRMN6P, U5 DRV8251ADDAR, U6 DRV8251ADDAR, U7 DRV8251ADDAR, U8 DRV8251ADDAR, U9 DRV8251ADDAR, X1 MKDSN1,5/8-5,08, X2 MKDSN1,5/2-5,08, X3 MKDSN1,5/2-5,08, X4 MKDSN1,5/8-5,08, X5 MKDSN1,5/8-5,08, X6 MKDSN1,5/2-5,08

Commit message: Hierarchical Schematic added
Parts:
- removed C1, C2, C3, C4, C5: 1uF, RTU_Agro_V4:C0603, symbol RTU_Agro_V4-eagle-import:C-EUC0603
- removed C10, C11, C12: 100nF, RTU_Agro_V4:C0603, symbol RTU_Agro_V4-eagle-import:C-EUC0603
- removed C13, C25: 4700uF, RTU_Agro_V4:E7,5-18, symbol RTU_Agro_V4-eagle-import:CPOL-EUE7.5-18
- removed C14, C15, C16, C17, C18, C19, C20, C21, C22, C23, C24, C6, C7: 0.1uF, RTU_Agro_V4:C0603, symbol RTU_Agro_V4-eagle-import:C-EUC0603
- removed C26: 100uF, RTU_Agro_V4:E2,5-6, symbol RTU_Agro_V4-eagle-import:CPOL-EUE2.5-6
- removed C8, C9: 20pF, RTU_Agro_V4:C0603, symbol RTU_Agro_V4-eagle-import:C-EUC0603
- removed D1, D2, D3, D4: ss54, RTU_Agro_V4:SMB, symbol RTU_Agro_V4-eagle-import:SCHOTTKY-DIODESMD
- removed IC1: STM32F103R8T6, RTU_Agro_V4:QFP50P1200X1200X160-64N, symbol RTU_Agro_V4-eagle-import:STM32F103R8T6
- removed J1: 520425-3, RTU_Agro_V4:520425-3, symbol RTU_Agro_V4-eagle-import:520425-3
- removed JMP1: 0R-JUMPB, RTU_Agro_V4:B0R-JMP, symbol RTU_Agro_V4-eagle-import:0R-JUMPB
- removed JP1: JP1, RTU_Agro_V4:JP1, symbol RTU_Agro_V4-eagle-import:JP1E
- removed L1: INDUCTOR_470, RTU_Agro_V4:INDUCTOR_470, symbol RTU_Agro_V4-eagle-import:INDUCTOR_470
- removed L2, L3: 100nH, RTU_Agro_V4:SM-1206, symbol RTU_Agro_V4-eagle-import:SM-1206
- removed LED1: Led1, RTU_Agro_V4:CHIPLED_0603, symbol RTU_Agro_V4-eagle-import:LEDCHIPLED_0603
- removed OK1, OK2, OK3, OK4: LTV816S, RTU_Agro_V4:DIL4-SMD, symbol RTU_Agro_V4-eagle-import:LTV816S
- removed R1: 10 mohm, RTU_Agro_V4:SMT-WAV, symbol RTU_Agro_V4-eagle-import:SMT-WAV
- removed R10, R11, R12, R13, R14, R16, R18, R22, R31, R32, R33, R34, R35, R36, R37, R38, R39, R44, R45: 10k, RTU_Agro_V4:R0603, symbol RTU_Agro_V4-eagle-import:R-EU_R0603
- removed R15, R17, R19, R21, R40, R41, R42, R43: 100, RTU_Agro_V4:R0603, symbol RTU_Agro_V4-eagle-import:R-EU_R0603
- removed R2, R3, R4, R47, R5: 1k, RTU_Agro_V4:R0603, symbol RTU_Agro_V4-eagle-import:R-EU_R0603
- removed R20: 120, RTU_Agro_V4:M1206, symbol RTU_Agro_V4-eagle-import:R-EU_M1206
- removed R23, R24, R25, R26, R27, R28, R29, R30: 1k, RTU_Agro_V4:M1206, symbol RTU_Agro_V4-eagle-import:R-EU_M1206
- removed R6: 3.3k, RTU_Agro_V4:M1206, symbol RTU_Agro_V4-eagle-import:R-EU_M1206
- removed R7: 50k, RTU_Agro_V4:RTRIM64W, symbol RTU_Agro_V4-eagle-import:R-TRIMM64W
- removed R8: 10k, RTU_Agro_V4:M1206, symbol RTU_Agro_V4-eagle-import:R-EU_M1206
- removed R9: 100k, RTU_Agro_V4:M1206, symbol RTU_Agro_V4-eagle-import:R-EU_M1206
- removed S1, S4: 1437566-4, RTU_Agro_V4:SW_1437566-4, symbol RTU_Agro_V4-eagle-import:1437566-4
- removed S2: SWS008, RTU_Agro_V4:SMS-008, symbol RTU_Agro_V4-eagle-import:SWS008
- removed SJ1: Sj1, RTU_Agro_V4:SJ, symbol RTU_Agro_V4-eagle-import:SJ
- removed U$1: MCP1727-3302E/SN, RTU_Agro_V4:SOIC127P599X175-8N, symbol RTU_Agro_V4-eagle-import:MCP1727-3302E/SN
- removed U1: XL4015, RTU_Agro_V4:CONV_XL4015, symbol RTU_Agro_V4-eagle-import:XL4015
- removed U10, U11, U12, U5, U6, U7, U8, U9: DRV8251ADDAR, RTU_Agro_V4:SOIC8_DDA_TEX, symbol RTU_Agro_V4-eagle-import:DRV8251ADDAR
- removed U13: PCF8574T, RTU_Agro_V4:SOIC127P1032X265-16N, symbol RTU_Agro_V4-eagle-import:PCF8574T
- removed U2: MAX3485ESA+, RTU_Agro_V4:SOIC127P600X175-8N, symbol RTU_Agro_V4-eagle-import:MAX3485ESA+
- removed U3: LTC2943IDD#TRPBF, RTU_Agro_V4:SON50P300X300X80-9N, symbol RTU_Agro_V4-eagle-import:LTC2943IDD#TRPBF
- removed U4: M24128-BRMN6P, RTU_Agro_V4:SOIC127P600X175-8N, symbol RTU_Agro_V4-eagle-import:M24128-BRMN6P
- removed X1, X4, X5: MKDSN1,5/8-5,08, RTU_Agro_V4:MKDSN1,5_8-5,08, symbol RTU_Agro_V4-eagle-import:MKDSN1,5/8-5,08
- removed X2, X3, X6: MKDSN1,5/2-5,08, RTU_Agro_V4:MKDSN1,5_2-5,08, symbol RTU_Agro_V4-eagle-import:MKDSN1,5/2-5,08
- removed XTAL1: CSM-7X-DU, RTU_Agro_V4:CSM-7X-DU, symbol RTU_Agro_V4-eagle-import:CSM-7X-DU
Other:
- added sheet Control (control.kicad_sch)
- added sheet Reeds switches (InSwitch.kicad_sch)
- added sheet Reguladores de voltaje (power_supply.kicad_sch)
- added sheet Valvula1 (OutValve.kicad_sch)
- added sheet Valvula2 (OutValve.kicad_sch)
- added sheet Valvula3 (OutValve.kicad_sch)
- added sheet Valvula4 (OutValve.kicad_sch)
- added sheet Valvula5 (OutValve.kicad_sch)
- added sheet Valvula6 (OutValve.kicad_sch)
- added sheet Valvula7 (OutValve.kicad_sch)
- added sheet Valvula8 (OutValve.kicad_sch)
- company: (none) -> ELECTROSHOP
- title: (none) -> RTU-Eneragro
